Commit message: add table

File: robots/abb_irb140.urdf.xacro (robot description, xacro)
@@ -1,11 +1,30 @@
 <?xml version="1.0"?>
 <robot xmlns:xacro="http://ros.org/wiki/xacro"
-       name="irb140" >
+  name="irb140" >
+  <xacro:arg name="load_table" default="false"/>
   <xacro:include filename="$(find irb140)/robots/irb140.xacro" />
   <xacro:include filename="$(find irb140)/robots/irb140.transmission.xacro"/>
+  <xacro:include filename="$(find irb140)/robots/table.urdf.xacro" />
   <xacro:property name="M_PI" value="3.1415926535897931" />
   <link name="world"/>
-  <xacro:irb140 parent="world">
-    <origin xyz="0 0 0" rpy="-1.57079632679 0 0" />
+  <joint name="world_joint" type="fixed">
+    <parent link="world"/>
+    <xacro:if value="$(arg load_table)">
+      <child link="table_link"/>
+      <origin xyz="0 0 0.845"/>
+    </xacro:if>
+    <xacro:unless value="$(arg load_table)">
+      <child link="fixation_link"/>
+      <origin xyz="0 0 0.0"/>
+    </xacro:unless>
+  </joint>
+  <!-- table -->
+  <xacro:if value="$(arg load_table)">
+    <xacro:table/>
+  </xacro:if>
+  <link name="fixation_link"/>
+  <!-- LWR -->
+  <xacro:irb140 parent="fixation_link">
+    <origin xyz="0.0 0 0.0" rpy="${-M_PI/2} 0 0" />
   </xacro:irb140>
   <gazebo>
@@ -14,4 +33,4 @@
     </plugin>
   </gazebo>
-   <xacro:irb140_transmission/>
+  <xacro:irb140_transmission/>
 </robot>

File: robots/irb140.xacro (robot description, xacro)
@@ -101,6 +101,6 @@
       xyz="0 0 1" />
     <limit
-      lower="${-M_PI}"
-      upper="${M_PI}"
+      lower="${-M_PI/4}"
+      upper="${M_PI/4}"
       effort="1000"
       velocity="200" />
@@ -170,6 +170,6 @@
       xyz="0 1 0" />
     <limit
-      lower="${-M_PI}"
-      upper="${M_PI}"
+      lower="${-M_PI/4}"
+      upper="${M_PI/2}"
       effort="1000"
       velocity="200" />
@@ -239,6 +239,6 @@
       xyz="0 1 0" />
     <limit
-      lower="${-M_PI}"
-      upper="${M_PI}"
+      lower="${-M_PI/4}"
+      upper="${M_PI/4}"
       effort="1000"
       velocity="200" />
@@ -377,6 +377,6 @@
       xyz="0 1 2.6185E-05" />
     <limit
-      lower="${-M_PI}"
-      upper="${M_PI}"
+      lower="${-M_PI/2}"
+      upper="${M_PI/2}"
       effort="1000"
       velocity="200" />
